File: hardware/kicad/sensor_hub.kicad_sch (KiCad schematic)
At the start: 0 parts

Commit message: hardware: generate KiCad 8 schematic skeleton (59 components)
hardware/tools/generate_schematic.py places all BOM components on an
A3 sheet with correct references, values, footprints, and DNP flags.
lib_symbols is empty — run Tools > Update Symbols from Library in
KiCad 8 to resolve. Then wire per hardware/docs/schematic.md.

Zone layout matches pcb_guidelines.md: analog left, EC (DNP) centre-
left, digital centre, PIR gate, relay right, connectors along bottom.

U3 (LMP91200) and U6 (VEML7700) may need manual symbol search if not
in the user's installed KiCad libraries.

Co-Authored-By: Claude Sonnet 4.6 <noreply@anthropic.com>
Parts:
- added C1, C10, C11, C12, C2, C3, C4, C5, C6, C7, C8, C9: 100nF, Capacitor_SMD:C_0603_1608Metric, symbol Device:C
- added C13, C14, C15, C16: 10uF, Capacitor_SMD:C_0805_2012Metric, symbol Device:C
- added C17, C18: 1uF, Capacitor_SMD:C_0603_1608Metric, symbol Device:C
- added D1: BAV99, Package_TO_SOT_SMD:SOT-23, symbol Diode:BAV99
- added D2: 1N4148W, Diode_SMD:D_SOD-123, symbol Device:D
- added HDR1: Debug-UART, Connector_PinHeader_2.54mm:PinHeader_1x04_P2.54mm_Vertical, symbol Connector_Generic:Conn_01x04
- added J1: 5-1634500-1, Connector_Coaxial:BNC_TE-Connectivity_1-1634500-1_Horizontal, symbol Connector_Coaxial:BNC_Jack
- added J2: Wago-DS18B20, TerminalBlock_Wago:TerminalBlock_Wago_2060-453_1x03_P5.00mm_Horizontal, symbol Connector_Generic:Conn_01x03
- added J3: Wago-DHT22, TerminalBlock_Wago:TerminalBlock_Wago_2060-453_1x03_P5.00mm_Horizontal, symbol Connector_Generic:Conn_01x03
- added J4: Wago-PIR, TerminalBlock_Wago:TerminalBlock_Wago_2060-453_1x03_P5.00mm_Horizontal, symbol Connector_Generic:Conn_01x03
- added J5: Wago-GP16, TerminalBlock_Wago:TerminalBlock_Wago_2060-453_1x03_P5.00mm_Horizontal, symbol Connector_Generic:Conn_01x03
- added J6: Wago-GP17, TerminalBlock_Wago:TerminalBlock_Wago_2060-453_1x03_P5.00mm_Horizontal, symbol Connector_Generic:Conn_01x03
- added J7: Wago-Relay, TerminalBlock_Wago:TerminalBlock_Wago_2060-453_1x03_P5.00mm_Horizontal, symbol Connector_Generic:Conn_01x03
- added J8: Phoenix-EC4pin, TerminalBlock_Phoenix:TerminalBlock_Phoenix_PT-1,5_4-3,5-H_1x04_P3.50mm_Horizontal, symbol Connector_Generic:Conn_01x04
- added J9: Phoenix-Power, TerminalBlock_Phoenix:TerminalBlock_Phoenix_PT-1,5_2-5,0-H_1x02_P5.00mm_Horizontal, symbol Connector_Generic:Conn_01x02
- added K1: SRD-05VDC-SL-C, Relay_THT:Relay_SPDT_Songle_SRD-xxVDC-SL-C, symbol Device:Relay_SPDT
- added Q1: BC817-40, Package_TO_SOT_SMD:SOT-23, symbol Transistor_BJT:BC817
- added Q2: BSS84PXUMA1, Package_TO_SOT_SMD:SOT-23, symbol Transistor_FET:BSS84
- added R1, R2: 10M, Resistor_SMD:R_0603_1608Metric, symbol Device:R
- added R10, R11: 4k7, Resistor_SMD:R_0603_1608Metric, symbol Device:R
- added R12, R13, R14, R8: 1k, Resistor_SMD:R_0603_1608Metric, symbol Device:R
- added R15, R16, R17, R19, R20, R21, R22, R7: 10k, Resistor_SMD:R_0603_1608Metric, symbol Device:R
- added R3, R4, R5, R6: 100k, Resistor_SMD:R_0603_1608Metric, symbol Device:R
- added U1: PicoW, MicrocontrollerBoard:RaspberryPi_PicoW, symbol MCU_RaspberryPi_RP2040:RaspberryPi_PicoW
- added U2: ADS1115IDGSR, Package_SO:VSSOP-10_3x3mm_P0.5mm, symbol Analog_ADC:ADS1115xDGS
- added U3: LMP91200SD/NOPB, Package_SO:SOIC-14_3.9x8.65mm_P1.27mm, symbol Sensor:LMP91200
- added U4: AD8603ARTZ-R2, Package_TO_SOT_SMD:SOT-23-5, symbol Amplifier_Operational:AD8603
- added U5: AP2112K-3.3TRG1, Package_TO_SOT_SMD:SOT-23-5, symbol Regulator_Linear:AP2112K-3.3
- added U6: VEML7700-TT, Package_DFN_QFN:DFN-6-1EP_2x2mm_P0.65mm_EP0.7x1.6mm, symbol Sensor_Optical:VEML7700
Other:
- note added: "ANALOG ZONE"
- note added: "After opening: Tools > Update Symbols from Library"
- note added: "CONNECTORS"
- note added: "DIGITAL ZONE"
- note added: "EC ZONE (DNP v1 — see schematic.md for v2 AD5933 plan)"
- note added: "PIR GATE"
- note added: "RELAY ZONE"
- note added: "U3 (LMP91200) + U6 (VEML7700) may need manual symbol search"
- note added: "Wire per hardware/docs/schematic.md"

Commit message: hardware: fix schematic generator component spacing
Components were overlapping after symbol library resolution in KiCad.
Rewrote COMPONENTS coordinates with ~2× more spacing: ICs get 30 mm+
clearance, connectors at 45 mm intervals, Pico W isolated at right,
EC DNP zone shifted to centre-left. Regenerated sensor_hub.kicad_sch.

Co-Authored-By: Claude Sonnet 4.6 <noreply@anthropic.com>
Other:
- note added: "EC ZONE (DNP v1 — AD5933 redesign for v2)"
- note removed: "EC ZONE (DNP v1 — see schematic.md for v2 AD5933 plan)"
