File: hardware/kicad/sensor_hub.kicad_sch (KiCad schematic)
At the start: 63 parts, among them J1 1-1478035-0, J10 Wago-Relay2, J11 Spare-GPIO, J2 Wago-DS18B20, J3 Wago-DHT22, J4 Wago-PIR, J5 Wago-GP16, J6 Wago-GP17, J7 Wago-Relay1, J8 Wago-EC4pin, J9 Wago-Power, K1 G2RL-1-E DC5, K2 G2RL-1-E DC5, Q1 BC817-40, Q2 BSS84PXUMA1, Q3 BC817-40, U1 Pico WH, U2 ADS1115IDGSR, U3 LMP91200SD/NOPB, U4 AD8603AUJZ, U5 AP2112K-3.3TRG1, U6 VEML7700-TT

Commit message: hardware: drop EC front-end, U6 under a light pipe with M2 holder holes
- U3 (LMP91200, EOL) and R15/R16/C3/C4/C5 removed from schematic, board and
  docs; GP13/GP14 now unused. NTC on J8 pins 3/4 unchanged.
- U6 (VEML7700) + C9 moved to the digital area below J11 (x 45 / y 73.45)
  for a light pipe to the lid; H5-H7 = 3x M2 NPTH on r = 7 mm for a
  3D-printed holder (the band only fits M2, not M2.5).
- autoroute: fixclear step narrows tracks that Freerouting leaves a few um
  under the clearance (0.25 -> 0.24 mm), routing unchanged.
- schematic.md / bom.csv / footprints.md / pcb_guidelines.md updated;
  J8/J9 no longer listed as Phoenix. fab/ re-exported.

Co-Authored-By: Claude Opus 5.5 (1M context) <noreply@anthropic.com>
Parts:
- removed C3, C4, C5: 100nF, Capacitor_SMD:C_0603_1608Metric, symbol Device:C
- removed R15, R16: 10k, Resistor_SMD:R_0603_1608Metric, symbol Device:R
- removed U3: LMP91200SD/NOPB, Package_SO:SOIC-14_3.9x8.7mm_P1.27mm, symbol Sensor:LMP91200
Connections:
- net EC_PWM_A: no longer names the net of U1.17 (GPIO13)
- net EC_PWM_B: no longer names the net of U1.19 (GPIO14)
- no-connect marks 9 -> 11
