File: hardware/kicad/sensor_hub.kicad_pcb (KiCad board)
At the start: 2 copper layers, 100 x 100 mm, 66 parts, among them J1 1-1478035-0, J10 Wago-Relay2, J11 Spare-GPIO, J2 Wago-DS18B20, J3 Wago-DHT22, J4 Wago-PIR, J5 Wago-GP16, J6 Wago-GP17, J7 Wago-Relay1, J8 Wago-EC4pin, J9 Wago-Power, K1 G2RL-1-E DC5, K2 G2RL-1-E DC5, Q1 BC817-40, Q2 BSS84PXUMA1, Q3 BC817-40, U1 Pico WH, U2 ADS1115IDGSR, U4 AD8603AUJZ, U5 AP2112K-3.3TRG1, U6 VEML7700-TT

Commit message: hardware: port labels above the terminals, 2601-1103 model
The W1-W5 / EC labels sat inside the terminal outlines and would be hidden
under the soldered Wago bodies. Now above them as 'J2  W1 DS18B20' etc.,
with the separate J2-J6/J8 reference fields hidden. fab/ re-exported.

Co-Authored-By: Claude Opus 5.5 <noreply@anthropic.com>
Claude-Session: https://claude.ai/code/session_01PDHupfXBxwLmo1MxXKJEdB
Other:
- board text added: "J2 W1 DS18B20"
- board text added: "J3 W2 DHT22"
- board text added: "J4 W3 PIR"
- board text added: "J5 W4 GP16"
- board text added: "J6 W5 GP17"
- board text added: "J8 EC W Y R B"
- board text removed: "EC W Y R B"
- board text removed: "W1 DS18B20"
- board text removed: "W2 DHT22"
- board text removed: "W3 PIR"
- board text removed: "W4 GP16"
- board text removed: "W5 GP17"

Commit message: hardware: drop EC front-end, U6 under a light pipe with M2 holder holes
- U3 (LMP91200, EOL) and R15/R16/C3/C4/C5 removed from schematic, board and
  docs; GP13/GP14 now unused. NTC on J8 pins 3/4 unchanged.
- U6 (VEML7700) + C9 moved to the digital area below J11 (x 45 / y 73.45)
  for a light pipe to the lid; H5-H7 = 3x M2 NPTH on r = 7 mm for a
  3D-printed holder (the band only fits M2, not M2.5).
- autoroute: fixclear step narrows tracks that Freerouting leaves a few um
  under the clearance (0.25 -> 0.24 mm), routing unchanged.
- schematic.md / bom.csv / footprints.md / pcb_guidelines.md updated;
  J8/J9 no longer listed as Phoenix. fab/ re-exported.

Co-Authored-By: Claude Opus 5.5 (1M context) <noreply@anthropic.com>
Parts:
- removed C3, C4, C5: 100nF, Capacitor_SMD:C_0603_1608Metric
- removed R15, R16: 10k, Resistor_SMD:R_0603_1608Metric
- added H5: MountingHole_2.2mm_M2, MountingHole:MountingHole_2.2mm_M2, F.Cu at (85.0, 106.5)
- added H6: MountingHole_2.2mm_M2, MountingHole:MountingHole_2.2mm_M2, F.Cu at (78.9, 117.0)
- added H7: MountingHole_2.2mm_M2, MountingHole:MountingHole_2.2mm_M2, F.Cu at (91.1, 117.0)
- moved U6 54.3 mm to (85.0, 114.3)
- moved C9 53.6 mm to (85.0, 116.7)
Connections:
- U1 pad 17: /EC_PWM_A -> (no net)
- U1 pad 19: /EC_PWM_B -> (no net)
Routing:
- net /I2C_SCL: track 38.2 -> 105.6 mm, vias 0 -> 3
- net /I2C_SDA: track 46.2 -> 102.5 mm
- net /GP19: track 101.4 -> 54.8 mm, vias 2 -> 3
- net /GP27: track 55.1 -> 96.1 mm, vias 0 -> 4
- net /EC_PWM_A: track 35.2 -> 0.00 mm, vias 1 -> 0
- net /EC_PWM_B: track 27.8 -> 0.00 mm, vias 1 -> 0
- net /PIR_EN_N: track 84.0 -> 57.6 mm, vias 3 -> 1
- net /3V3_DIG: track 296.2 -> 272.7 mm, vias 3 -> 1
- net /UART_RX: track 94.2 -> 113.1 mm, vias 0 -> 4
- net /RELAY1_DRV: track 45.2 -> 61.7 mm, vias 2 -> 1
- net /W5_SIG: track 83.7 -> 69.9 mm, vias 3 -> 1
- net /3V3_ANA: track 106.0 -> 116.1 mm
- net /GP7: track 33.6 -> 43.7 mm, vias 0 -> 1
- net /GP6: track 40.0 -> 49.8 mm
- net /GND_ANA: track 165.2 -> 155.8 mm, vias 1 -> 2
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